Commit message: Update README and launch files for improved simulation setup; add IMU frame and sensor configurations

File: models/base_model.urdf (robot description, URDF)
Before this commit: robot default_robot, 6 links, 5 joints
Links:
- added link imu_frame, mass 0.01; visual box size=0.01 0.01 0.01
Joints:
- added joint imu_joint: type fixed, parent base_link, child imu_frame, origin xyz=0 0 0.04 rpy=0 0 0

Commit message: Add grid visualization to RViz configuration and adjust IMU joint orientation

File: models/base_model.urdf (robot description, URDF)
Before this commit: robot default_robot, 7 links, 6 joints
Joints:
- joint right_wheel_joint: origin xyz=-0.05 -0.06 -0.035 rpy=1.5707 0 0 -> xyz=-0.05 -0.06 -0.035 rpy=-1.5707 0 0
